File: KiCad/Xeltri/STM32.kicad_sch (KiCad schematic)
At the start: 38 parts, among them U5 STM32H745XIHx

Commit message: Sync KiCad layout and schematics from the portable work-tree.
Co-authored-by: Cursor <cursoragent@cursor.com>
Parts:
- added C82: 100nF, Capacitor_SMD:C_0402_1005Metric, symbol Device:C
- added R61: 10K, Resistor_SMD:R_0402_1005Metric, symbol Device:R
Connections:
- net GND: now also C82.1, R61.1
- net at C51.1, U5.D17 (VCAP), U5.U11 (VCAP): now also C50.2, U5.A7 (VCAP)
- net at U5.E8 (BOOT0): now also R61.2
- net at U5.K1 (NRST): now also C82.2
