File: KiCad/Xeltri/STM32.kicad_sch (KiCad schematic)
At the start: 40 parts, among them U5 STM32H745XIHx

Commit message: Lay out STM32 power decoupling and add USB FS plus 24 V CIN ceramics.
USB VDD33/VDD50 share local 100 nF + 1 µF on 3.3 V; VBAT keeps a local 100 nF until the cell and diode are placed.

Co-authored-by: Cursor <cursoragent@cursor.com>
Parts:
- added C85: 100nF/16V, Capacitor_SMD:C_0402_1005Metric, symbol Device:C
- added C86: 1uF/25V, Capacitor_SMD:C_0402_1005Metric, symbol Device:C
Connections:
- net +3.3V: now also C85.1, C86.1
- net GND: now also C85.2, C86.2
Other:
- moved on the sheet: C50, C52, C53, C54, C55, C56, C57, C58, C59, C60, C61, C62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
