File: KiCad/Xeltri/Xeltri.kicad_pcb (KiCad board)
At the start: 6 copper layers, 100 x 100 mm, 188 parts, among them J1 PJ-035DH, J2 877159106, J3 HR911105A_C12074, Q1 AOD407, U1 XC7A35T-CSG325, U10 SY8843QWC, U11 RT9013-18GB, U12 RT9013-12GB, U13 TPS22966DPUR, U14 TPS22966DPUR, U15 TPS22966DPUR, U16 TPS22966DPUR, U17 CH334P, U2 V851S, U3 TPS56637RPAR, U4 TPS56637RPAR, U5 STM32H745XIHx, U6 RTL8201F-VB-CG, U7 SY8843QWC, U8 SY8843QWC, U9 SY8843QWC, Y1 25Mhz

Commit message: Sync KiCad layout and schematics from the portable work-tree.
Co-authored-by: Cursor <cursoragent@cursor.com>
Parts:
- removed R59: 0R, Resistor_SMD:R_0402_1005Metric
- added C82: 100nF, Capacitor_SMD:C_0402_1005Metric, F.Cu at (129.2, 54.0)
- added R61: 10K, Resistor_SMD:R_0402_1005Metric, F.Cu at (129.2, 52.0)
- C13, C3: value 0.1uF -> 100nF
- moved C80 7.92 mm to (132.3, 69.9)
- moved C81 7.92 mm to (132.3, 71.8)
- moved L1 0.97 mm to (119.6, 128.0)
- moved R39 0.73 mm to (121.4, 123.5)
- moved C4 0.54 mm to (124.2, 130.5)
Connections:
- C29 pad 1: /power/SY8843_3.3V_OUT -> +3.3V
- C4 pad 2: Net-(C4-Pad2) -> Net-(U3-SW)
- C45 pad 1: /power/SY8843_3.3V_OUT -> +3.3V
- C51 pad 1: Net-(C51-Pad1) -> Net-(C50-Pad2)
- L3 pad 2: /power/SY8843_3.3V_OUT -> +3.3V
- R31 pad 1: /power/SY8843_3.3V_OUT -> +3.3V
- R36 pad 1: /power/SY8843_3.3V_OUT -> +3.3V
- R45 pad 1: /power/SY8843_3.3V_OUT -> +3.3V
- R46 pad 1: /power/SY8843_3.3V_OUT -> +3.3V
- R48 pad 1: /power/SY8843_3.3V_OUT -> +3.3V
- U13 pad 1: /power/SY8843_3.3V_OUT -> +3.3V
- U13 pad 13: +3.3V -> Net-(U13-VOUT1-Pad13)
- U13 pad 14: +3.3V -> Net-(U13-VOUT1-Pad13)
- U13 pad 2: /power/SY8843_3.3V_OUT -> +3.3V
- U13 pad 4: /power/SY8843_3.3V_OUT -> +3.3V
- U5 pad D17: Net-(C51-Pad1) -> Net-(C50-Pad2)
- U5 pad E8: unconnected-(U5-BOOT0-PadE8) -> Net-(U5-BOOT0)
- U5 pad K1: unconnected-(U5-NRST-PadK1) -> Net-(U5-NRST)
- U5 pad U11: Net-(C51-Pad1) -> Net-(C50-Pad2)
- U7 pad 2: /power/SY8843_3.3V_OUT -> +3.3V
Routing:
- net Net-(U3-SW): track 6.64 -> 3.19 mm
- net +5V: track 22.8 -> 20.2 mm
- net Net-(C4-Pad2): track 1.04 -> 0.00 mm
- added copper zone on F.Cu, net Net-(U3-SW)
