File: KiCad/Xeltri/Xeltri.kicad_pcb (KiCad board)
At the start: 6 copper layers, 100 x 100 mm, 189 parts, among them J1 PJ-035DH, J2 877159106, J3 HR911105A_C12074, Q1 AOD407, U1 XC7A35T-CSG325, U10 SY8843QWC, U11 RT9013-18GB, U12 RT9013-12GB, U13 TPS22966DPUR, U14 TPS22966DPUR, U15 TPS22966DPUR, U16 TPS22966DPUR, U17 CH334P, U2 V851S, U3 TPS56637RPAR, U4 TPS56637RPAR, U5 STM32H745XIHx, U6 RTL8201F-VB-CG, U7 SY8843QWC, U8 SY8843QWC, U9 SY8843QWC, Y1 25Mhz

Commit message: Update KiCad project files: enhance .gitignore for sensitive data, refine component properties in schematics, and remove obsolete MCU configuration file. Added LCSC part numbers and datasheets for various components.
Parts:
- removed R60: 0R, Resistor_SMD:R_0402_1005Metric
- C1, C11, C12, C2: value 10uF -> 10uF/50V; footprint Capacitor_SMD:C_1210_3225Metric -> Capacitor_SMD:C_1206_3216Metric
- C13, C14, C3, C4: value 100nF -> 100nF/50V
- C15, C5: value 100pF -> 100pF/50V
- C16, C17, C18, C29, C31, C32, C34, C35, C37, C38, C40, C45, C46, C47, C48, C6, C7, C8, C9: value 22uF -> 22uF/25V
- C20, C21: value 10nF -> 10nF/50V
- C22, C25, C27, C30, C33, C36, C39, C49, C52, C53, C55, C56, C57, C58, C59, C60, C61, C62, C63, C64, C65, C66, C67, C68, C69, C70, C71, C72, C73, C75, C79, C80, C81, C82: value 100nF -> 100nF/16V
- C23, C24: value 15pF -> 15pF/50V
- C26, C28: value 10uF -> 10uF/6.3V
- C41, C42, C43, C44, C54, C74: value 1uF -> 1uF/25V
- C50, C51: value 2.2uF -> 2.2uF/6.3V
- C76, C77, C78: value 4.7uF -> 4.7uF/25V
- moved C35 5.38 mm to (114.1, 95.0)
- moved C36 5.38 mm to (115.8, 95.1)
- moved C37 5.38 mm to (119.3, 91.6)
- moved C47 5.38 mm to (116.6, 90.9)
- moved L5 5.38 mm to (118.6, 95.9)
- moved R37 5.38 mm to (121.1, 93.1)
- moved R47 5.38 mm to (121.1, 91.1)
- moved R54 5.38 mm to (114.3, 92.6)
- moved U9 5.38 mm to (117.1, 93.1)
- moved C39 2.93 mm to (120.2, 84.5)
- moved C40 2.93 mm to (123.7, 80.9)
- moved L6 2.93 mm to (122.9, 85.0)
- moved R55 2.93 mm to (118.7, 81.7)
- moved U10 2.93 mm to (121.4, 82.5)
- moved C38 2.93 mm to (118.4, 84.3)
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Connections:
- C14 pad 2: Net-(C14-Pad2) -> Net-(U4-SW)
- U2 pad 89: unconnected-(U2-EPAD-Pad89) -> GND
Routing:
- net Net-(U4-SW): track 6.51 -> 4.32 mm
- net Net-(C14-Pad2): track 0.97 -> 0.00 mm
- net unconnected-(U2-EPAD-Pad89): vias 25 -> 0
- net GND: vias 193 -> 219
- added copper zone on F.Cu, net +3.3V
- added copper zone on F.Cu, net Net-(U4-SW)
- removed copper zone on F.Cu, net /power/SY8843_3.3V_OUT
