File: KiCad/Xeltri/FPGA.kicad_sch (KiCad schematic)
At the start: 1 part, among them U1 XC7A35T-CSG325

Commit message: Match the six-layer stackup to JLC06161H-3313 and update FPGA power wiring.
Co-authored-by: Cursor <cursoragent@cursor.com>
Parts:
- added C100, C101, C102, C103, C104, C105, C106, C107, C108, C109, C110, C111, C112, C113, C114, C115, C116, C117, C118, C119, C120, C121, C122, C123, C124, C125, C126, C127, C128, C129, C130, C131, C132, C133, C134, C135, C136, C137, C138, C139, C140, C141, C142, C143, C144, C87, C88, C89, C90, C91, C92, C93, C94, C95, C96, C97, C98, C99: 470nF, Capacitor_SMD:C_0402_1005Metric, symbol Device:C
- added FB3: 600R@100M, Inductor_SMD:L_0402_1005Metric, symbol Device:FerriteBead
- added R59: 100R, Resistor_SMD:R_0402_1005Metric, symbol Device:R
Connections:
- net GND: now also U1.J9 (GNDADC_0), C100.2, C101.2, C102.2, C103.2, C104.2, C105.2, C106.2, C107.2, C108.2, C109.2, C110.2, C111.2, C112.2, C113.2, C114.2, C115.2, C116.2, C117.2, C118.2, C119.2, C120.2, C121.2, C122.2, C123.2, C124.2, C125.2, C126.2, C127.2, C128.2, C129.2, C130.2, C131.2, C132.2, C133.2, C134.2, C135.2, C136.2, C137.2, C138.2, C139.2, C140.2, C141.2, C142.2, C143.2, C144.2, C87.2, C88.2, C89.2, C90.2, C91.2, C92.2, C93.2, C94.2, C95.2, C96.2, C97.2, C98.2, C99.2
- net FPGA_3.3V: now reaches U1.E10 (VCCO_0)
- net FPGA_3.3V: now also U1.A16 (VCCO_15), U1.B13 (VCCO_15), U1.C10 (VCCO_15), U1.D17 (VCCO_15), U1.E14 (VCCO_15), U1.G18 (VCCO_15), U1.H15 (VCCO_15), U1.L16 (VCCO_14), U1.L6 (VCCO_34), U1.M3 (VCCO_34), U1.P17 (VCCO_14), U1.P7 (VCCO_34), U1.R10 (VCCO_0), U1.R14 (VCCO_14), U1.R4 (VCCO_34), U1.T1 (VCCO_34), U1.T11 (VCCO_14), U1.U18 (VCCO_14), U1.U8 (VCCO_14), U1.V15 (VCCO_14), U1.V5 (VCCO_34), C108.1, C109.1, C110.1, C111.1, C112.1, C113.1, C114.1, C115.1, C116.1, C117.1, C118.1, C119.1, C120.1, C121.1, C122.1, C123.1, C124.1, C125.1, C126.1, C127.1, C128.1, C129.1
- net FPGA_1V2: now reaches U1.A2 (MGTAVTT)
- net FPGA_1V2: now also U1.C1 (MGTAVTT), U1.E1 (MGTAVTT), U1.F3 (MGTAVTT), U1.G2 (MGTAVTT), C136.1, C137.1, C138.1, C139.1, C140.1, R59.2
- net at U1.A6 (MGTRREF_216): now also R59.1
- net FPGA_MGTAVCC: now reaches U1.B4 (MGTAVCC)
- net FPGA_MGTAVCC: now also U1.C5 (MGTAVCC), U1.E5 (MGTAVCC), U1.F5 (MGTAVCC), C141.1, C142.1, C143.1, C144.1, FB3.2
- net FPGA_1V8: now reaches U1.E11 (VCCBATT_0)
- net FPGA_1V8: now also U1.G12 (VCCAUX), U1.H13 (VCCAUX), U1.J10 (VCCADC_0), U1.K13 (VCCAUX), U1.M13 (VCCAUX), U1.P13 (VCCAUX), C130.1, C131.1, C132.1, C133.1, C134.1, C135.1
- net FPGA_1V0: now reaches U1.F11 (VCCBRAM)
- net FPGA_1V0: now also U1.F7 (VCCINT), U1.F9 (VCCINT), U1.G10 (VCCBRAM), U1.G8 (VCCINT), U1.H11 (VCCBRAM), U1.H7 (VCCINT), U1.H9 (VCCINT), U1.J12 (VCCINT), U1.J8 (VCCINT), U1.K11 (VCCINT), U1.K7 (VCCINT), U1.L12 (VCCINT), U1.L8 (VCCINT), U1.M11 (VCCINT), U1.M7 (VCCINT), U1.N10 (VCCINT), U1.N12 (VCCINT), U1.N8 (VCCINT), U1.P11 (VCCINT), U1.P9 (VCCINT), C100.1, C101.1, C102.1, C103.1, C104.1, C105.1, C106.1, C107.1, C87.1, C88.1, C89.1, C90.1, C91.1, C92.1, C93.1, C94.1, C95.1, C96.1, C97.1, C98.1, C99.1, FB3.1
Other:
- moved on the sheet: U1A, U1B, U1C, U1D, U1E, U1F
