File: analysis/backup_sch_mlcc/Expansion_Port.kicad_sch (KiCad schematic)
At the start: 35 parts, among them J2 877159106, J3 HR911105A_C12074, U17 CH334P, U6 RTL8201F-VB-CG, Y1 25Mhz

Commit message: Update KiCad project files: enhance .gitignore for sensitive data, refine component properties in schematics, and remove obsolete MCU configuration file. Added LCSC part numbers and datasheets for various components.
Parts:
- C19: LCSC Part C1523 -> (none)
- C20, C21: value 10nF/50V -> 10nF; LCSC Part C15195 -> (none)
- C22, C25, C27: value 100nF/16V -> 100nF; LCSC Part C1525 -> (none)
- C23, C24: value 15pF/50V -> 15pF; LCSC Part C1548 -> (none)
- C26, C28: value 10uF/6.3V -> 10uF; LCSC Part C15525 -> (none)
Changed lines of the file:
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@@
 			)
 		)
-		(property "Value" "15pF/50V"
+		(property "Value" "15pF"
 			(at 77.47 218.4399 0)
 			(effects
@@
 			)
 		)
-		(property "Datasheet" "https://jlcpcb.com/partdetail/FH-0402CG150J500NT/C1548"
+		(property "Datasheet" "~"
 			(at 73.66 217.17 0)
 			(effects
@@
 			)
 		)
-		(property "LCSC Part" "C1548"
-			(at 0 0 0)
-			(effects
-				(font
-					(size 1.27 1.27)
-				)
-				(hide yes)
-			)
-		)
 		(pin "1"
 		)
@@
 			)
 		)
-		(property "Value" "100nF/16V"
+		(property "Value" "100nF"
 			(at 118.11 210.058 90)
 			(effects
@@
 			)
 		)
-		(property "Datasheet" "https://jlcpcb.com/partdetail/Samsung-CL05B104KO5NNNC/C1525"
+		(property "Datasheet" "~"
 			(at 119.38 205.74 0)
 			(effects
@@
 			)
 		)
-		(property "LCSC Part" "C1525"
-			(at 0 0 0)
-			(effects
-				(font
-					(size 1.27 1.27)
-				)
-				(hide yes)
-			)
-		)
 		(pin "1"
 		)
@@
 			)
 		)
-		(property "Datasheet" "https://jlcpcb.com/partdetail/FH-0402B102K500NT/C1523"
+		(property "Datasheet" "~"
 			(at 284.48 260.35 0)
 			(effects
@@
 			)
 		)
-		(property "LCSC Part" "C1523"
-			(at 0 0 0)
-			(effects
-				(font
-					(size 1.27 1.27)
-				)
-				(hide yes)
-			)
-		)
 		(pin "1"
 		)
@@
 			)
 		)
-		(property "Value" "100nF/16V"
+		(property "Value" "100nF"
 			(at 85.09 246.38 90)
 			(effects
@@
 			)
 		)
-		(property "Datasheet" "https://jlcpcb.com/partdetail/Samsung-CL05B104KO5NNNC/C1525"
+		(property "Datasheet" "~"
 			(at 85.09 251.46 0)
 			(effects
@@
 			)
 		)
-		(property "LCSC Part" "C1525"
-			(at 0 0 0)
-			(effects
-				(font
-					(size 1.27 1.27)
-				)
-				(hide yes)
-			)
-		)
 		(pin "1"
 		)
@@
 			)
 		)
-		(property "Value" "10nF/50V"
+		(property "Value" "10nF"
 			(at 311.15 239.776 90)
 			(effects
@@
 			)
 		)
-		(property "Datasheet" "https://jlcpcb.com/partdetail/Samsung-CL05B103KB5NNNC/C15195"
+		(property "Datasheet" "~"
 			(at 311.15 243.84 0)
 			(effects
@@
 			)
 		)
-		(property "LCSC Part" "C15195"
-			(at 0 0 0)
-			(effects
-				(font
-					(size 1.27 1.27)
-				)
-				(hide yes)
-			)
-		)
 		(pin "1"
 		)
@@
 			)
 		)
-		(property "Value" "10nF/50V"
+		(property "Value" "10nF"
 			(at 311.15 249.936 90)
 			(effects
@@
 			)
 		)
-		(property "Datasheet" "https://jlcpcb.com/partdetail/Samsung-CL05B103KB5NNNC/C15195"
+		(property "Datasheet" "~"
 			(at 311.15 254 0)
 			(effects
@@
 			)
 		)
-		(property "LCSC Part" "C15195"
-			(at 0 0 0)
-			(effects
-				(font
-					(size 1.27 1.27)
-				)
-				(hide yes)
-			)
-		)
 		(pin "1"
 		)
@@
 			)
 		)
-		(property "Value" "15pF/50V"
+		(property "Value" "15pF"
 			(at 105.41 218.4399 0)
 			(effects
@@
 			)
 		)
-		(property "Datasheet" "https://jlcpcb.com/partdetail/FH-0402CG150J500NT/C1548"
+		(property "Datasheet" "~"
 			(at 101.6 217.17 0)
 			(effects
@@
 			)
 		)
-		(property "LCSC Part" "C1548"
-			(at 0 0 0)
-			(effects
-				(font
-					(size 1.27 1.27)
-				)
-				(hide yes)
-			)
-		)
 		(pin "1"
 		)
@@
 			)
 		)
-		(property "Value" "100nF/16V"
+		(property "Value" "100nF"
 			(at 64.77 303.5299 0)
 			(effects
@@
 			)
 		)
-		(property "Datasheet" "https://jlcpcb.com/partdetail/Samsung-CL05B104KO5NNNC/C1525"
+		(property "Datasheet" "~"
 			(at 60.96 302.26 0)
 			(effects
@@
 			)
 		)
-		(property "LCSC Part" "C1525"
-			(at 0 0 0)
-			(effects
-				(font
-					(size 1.27 1.27)
-				)
-				(hide yes)
-			)
-		)
 		(pin "1"
 		)
@@
 			)
 		)
-		(property "Value" "10uF/6.3V"
+		(property "Value" "10uF"
 			(at 52.07 303.5299 0)
 			(effects
@@
 			)
 		)
-		(property "Datasheet" "https://jlcpcb.com/partdetail/Samsung-CL05A106MQ5NUNC/C15525"
+		(property "Datasheet" "~"
 			(at 48.26 302.26 0)
 			(effects
@@
 			)
 		)
-		(property "LCSC Part" "C15525"
-			(at 0 0 0)
-			(effects
-				(font
-					(size 1.27 1.27)
-				)
-				(hide yes)
-			)
-		)
 		(pin "1"
 		)
@@
 			)
 		)
-		(property "Value" "10uF/6.3V"
+		(property "Value" "10uF"
 			(at 39.37 303.5299 0)
 			(effects
@@
 			)
 		)
-		(property "Datasheet" "https://jlcpcb.com/partdetail/Samsung-CL05A106MQ5NUNC/C15525"
+		(property "Datasheet" "~"
 			(at 35.56 302.26 0)
 			(effects
@@
 			(effects
 				(font
-					(size 1.27 1.27)
-				)
-				(hide yes)
-			)
-		)
-		(property "LCSC Part" "C15525"
-			(at 0 0 0)
-			(effects
-				(font
