File: analysis/backup_sch_mlcc/STM32.kicad_sch (KiCad schematic)
At the start: 40 parts, among them U5 STM32H745XIHx

Commit message: Update KiCad project files: enhance .gitignore for sensitive data, refine component properties in schematics, and remove obsolete MCU configuration file. Added LCSC part numbers and datasheets for various components.
Parts:
- C49, C52, C53, C55, C56, C57, C58, C59, C60, C61, C62, C63, C64, C65, C66, C67, C68, C69, C70, C71, C72, C73, C75, C79, C80, C81, C82: value 100nF/16V -> 100nF; LCSC Part C1525 -> (none)
- C50, C51: value 2.2uF/6.3V -> 2.2uF; LCSC Part C12530 -> (none)
- C54, C74: value 1uF/25V -> 1uF; LCSC Part C52923 -> (none)
- C76, C77, C78: value 4.7uF/25V -> 4.7uF; LCSC Part C1779 -> (none)
