File: analysis/backup_sch_mlcc/power.kicad_sch (KiCad schematic)
At the start: 110 parts, among them J1 PJ-035DH, Q1 AOD407, U10 SY8843QWC, U11 RT9013-18GB, U12 RT9013-12GB, U13 TPS22966DPUR, U14 TPS22966DPUR, U15 TPS22966DPUR, U16 TPS22966DPUR, U3 TPS56637RPAR, U4 TPS56637RPAR, U7 SY8843QWC, U8 SY8843QWC, U9 SY8843QWC

Commit message: Update KiCad project files: enhance .gitignore for sensitive data, refine component properties in schematics, and remove obsolete MCU configuration file. Added LCSC part numbers and datasheets for various components.
Parts:
- C1, C11, C12, C2: value 10uF/50V -> 10uF; footprint Capacitor_SMD:C_1206_3216Metric -> Capacitor_SMD:C_1210_3225Metric; LCSC Part C13585 -> (none)
- C13, C3: value 100nF/50V -> 100nF; LCSC Part C49678 -> (none)
- C14, C4: value 100nF/50V -> 100nF; LCSC Part C307331 -> (none)
- C15, C5: value 100pF/50V -> 100pF; LCSC Part C1546 -> (none)
- C16, C17, C18, C29, C31, C32, C34, C35, C37, C38, C40, C45, C46, C47, C48, C6, C7, C8, C9: value 22uF/25V -> 22uF; LCSC Part C45783 -> (none)
- C30, C33, C36, C39: value 100nF/16V -> 100nF; LCSC Part C1525 -> (none)
- C41, C42, C43, C44: value 1uF/25V -> 1uF; LCSC Part C52923 -> (none)
